Commit message: .

File: diff_summer_robot_description/urdf/diff_summer_robot.urdf (robot description, URDF)
Before this commit: robot diff_summer_robot, 1 links, 0 joints
Links:
- added link second_link; visual cylinder length=0.1 radius=0.1
- added link third_link; visual box size=0.1 0.1 0.1
- link base_link: geometry visual box size=0.6 0.4 0.2
Joints:
- added joint base_to_second: type continuous, parent base_link, child second_link, origin xyz=0.0 0 0.2 rpy=0 0 0, axis 0.0 0.0 1, limit lower=-1.57 upper=1.57 effort=10.0 velocity=3.14
- added joint second_to_third: type prismatic, parent second_link, child third_link, origin xyz=0.0 0 0.1 rpy=0 0 0, axis 1 0.0 0.0, limit lower=0.0 upper=0.2 effort=10.0 velocity=0.05
