Commit message: first commit workspace ROS 2

File: diff_test_description/urdf/common_properties.xacro (robot description, xacro)
@@ -10,3 +10,24 @@
         <color rgba="0.0 .0 0.0 1.0"/>
     </material>
+    <xacro:macro name="box_inertia" params="l w h m o_xyz o_rpy">
+        <inertial>
+            <origin xyz="${o_xyz}" rpy="${o_rpy}"/>
+            <mass value="${m}"/>
+            <inertia ixx="${m*(w*w+h*h)/12.0}" ixy="0.0" ixz="0.0" iyy="${m*(l*l+h*h)/12.0}" iyz="0.0" izz="${m*(w*w+l*l)/12.0}"/>
+        </inertial>
+    </xacro:macro>
+    <xacro:macro name="cylinder_inertia" params="r l m o_xyz o_rpy">
+        <inertial>
+            <origin xyz="${o_xyz}" rpy="${o_rpy}"/>
+            <mass value="${m}"/>
+            <inertia ixx="${m * (3.0 * r * r + l * l) / 12.0}" ixy="0.0" ixz="0.0" iyy="${m*(l*l+3*r*r)/12.0}" iyz="0.0" izz="${m * r * r / 2.0}"/>
+        </inertial>
+    </xacro:macro>
+    <xacro:macro name="sphere_inertia" params="r m o_xyz o_rpy">
+        <inertial>
+            <origin xyz="${o_xyz}" rpy="${o_rpy}"/>
+            <mass value="${m}"/>
+            <inertia ixx="${2.0 * m * r * r / 5.0}" ixy="0.0" ixz="0.0" iyy="${2.0 * m * r * r / 5.0}" iyz="0.0" izz="${2.0 * m * r * r / 5.0}"/>
+        </inertial>
+    </xacro:macro>
 </robot>

File: diff_test_description/urdf/diff_sumer_robot_tutor.xacro (robot description, xacro)
@@ -3,3 +3,6 @@
     <xacro:include filename="$(find diff_test_description)/urdf/common_properties.xacro"/>
     <xacro:include filename="$(find diff_test_description)/urdf/mobile_base.xacro"/>
+    <xacro:include filename="$(find diff_test_description)/urdf/mobile_base_gazebo.xacro"/>
+    <xacro:include filename="$(find diff_test_description)/urdf/camera.xacro"/>
+    <xacro:include filename="$(find diff_test_description)/urdf/lidar.xacro"/>
 </robot>

File: diff_test_description/urdf/mobile_base.xacro (robot description, xacro)
@@ -8,4 +8,5 @@
     <xacro:macro name="wheel_link" params="prefix radius length">
         <link name="${prefix}_wheel_link">
+        <xacro:cylinder_inertia r="${radius}" l="${length}" m="1.0" o_xyz="0.0 0.0 0.0" o_rpy="${pi / 2.0} 0.0 0.0"/>
         <visual>
             <geometry>
@@ -15,19 +16,33 @@
             <material name="grey"/>
         </visual>
+        <collision>
+            <origin xyz="0.0 0.0 0.0" rpy="${pi / 2.0} 0.0 0.0"/>
+            <geometry>
+                <sphere radius="${wheel_radius}"/>
+            </geometry>
+        </collision>
     </link>
     </xacro:macro>
-    <link name="base_footprint"></link>
+    <link name="base_footprint"/>
     <link name="base_link">
+        <xacro:box_inertia l="${base_length}" w="${base_width}" h="${base_height}" m="5.0" o_xyz="0.0 0.0 ${base_height/2.0}" o_rpy="0.0 0.0 0.0"/>
         <visual>
             <geometry>
                 <box size="${base_length} ${base_width} ${base_height}"/>
             </geometry>
-            <origin xyz="0.0 0.0 ${wheel_radius}" rpy="0.0 0.0 0.0"/>
+            <origin xyz="0.0 0.0 ${base_height/2.0}" rpy="0.0 0.0 0.0"/>
             <material name="blue"/>
         </visual>
+        <collision>
+            <origin xyz="0.0 0.0 ${base_height/2.0}" rpy="0.0 0.0 0.0"/>
+            <geometry>
+                <box size="${base_length} ${base_width} ${base_height}"/>
+            </geometry>
+        </collision>
     </link>
     <xacro:wheel_link prefix="right" radius="${wheel_radius}" length="${wheel_length}"/>
     <xacro:wheel_link prefix="left" radius="${wheel_radius}" length="${wheel_length}"/>
     <link name="caster_wheel_link">
+        <xacro:sphere_inertia r="${wheel_radius / 2}" m="0.5" o_xyz="0.0 0.0 0.0" o_rpy="0.0 0.0 0.0"/>
         <visual>
             <geometry>
@@ -37,4 +52,10 @@
             <material name="grey"/>
         </visual>
+        <collision>
+                <origin xyz="0.0 0.0 0.0" rpy="0.0 0.0 0.0"/>
+                <geometry>
+                    <sphere radius="${wheel_radius / 2}"/>
+                </geometry>
+            </collision>
     </link>
     <joint name="footprint_to_base_joint" type="fixed">
@@ -55,5 +76,5 @@
         <axis xyz="0.0 1.0 0.0"/>
     </joint>
-    <joint name="base_to_caster_wheel" type="continuous">
+    <joint name="base_to_caster_wheel" type="fixed">
         <parent link="base_link"/>
         <child link="caster_wheel_link"/>
